Commit message: Update

File: marrtinorobot2_description/urdf/2wd_properties.urdf.xacro (robot description, xacro)
@@ -5,5 +5,5 @@
   <xacro:property name="base_height" value="0.003" />
   <xacro:property name="base_mass" value="1" />
-  <xacro:property name="wheel_radius" value="0.05" />
+  <xacro:property name="wheel_radius" value="0.045" />
   <xacro:property name="wheel_width" value="0.01" />
   <xacro:property name="wheel_pos_x" value="0.0" />
@@ -12,5 +12,5 @@
   <xacro:property name="wheel_mass" value=".1" />
   <xacro:property name="wheel_torque" value="20" />
-  <xacro:property name="front_caster_wheel" value="false" />
+  <xacro:property name="front_caster_wheel" value="true" />
   <xacro:property name="rear_caster_wheel" value="true" />
   <xacro:property name="laser_pose">

File: marrtinorobot2_description/urdf/mech/caster_wheel.urdf.xacro (robot description, xacro)
@@ -3,9 +3,7 @@
   <xacro:macro name="caster_wheel" params="side mass base_length wheel_radius wheel_pos_z">
     <xacro:property name="caster_wheel_radius" value="${(wheel_radius - wheel_pos_z) / 2}" />
-    <!--
     <xacro:if value="${side == 'front'}">
         <xacro:property name="caster_wheel_x" value="${(base_length / 2) - caster_wheel_radius}" />
     </xacro:if>
-    -->
     <xacro:if value="${side == 'rear'}">
         <xacro:property name="caster_wheel_x" value="${-(base_length / 2) + caster_wheel_radius}" />

File: marrtinorobot2_description/urdf/robots/2wd.urdf.xacro (robot description, xacro)
@@ -35,5 +35,4 @@
     mass="${wheel_mass}"
   />
- <!--
   <xacro:if value="${front_caster_wheel}">
     <xacro:caster_wheel
@@ -45,5 +44,4 @@
     />
   </xacro:if>
--->
   <xacro:if value="${rear_caster_wheel}">
     <xacro:caster_wheel

Commit message: MarrtinoRobot ROS 2

File: marrtinorobot2_description/urdf/2wd_properties.urdf.xacro (robot description, xacro)
@@ -15,5 +15,5 @@
   <xacro:property name="rear_caster_wheel" value="true" />
   <xacro:property name="laser_pose">
-    <origin xyz="0.12 0 0.33" rpy="0 0 0"/>
+    <origin xyz="0.12 0 0.13" rpy="0 0 0"/>
   </xacro:property>
   <xacro:property name="depth_sensor_pose">

Commit message: MARRtino Robot ROS2

File: marrtinorobot2_description/urdf/2wd_properties.urdf.xacro (robot description, xacro)
@@ -1,19 +1,19 @@
 <?xml version="1.0"?>
 <robot xmlns:xacro="http://ros.org/wiki/xacro">
-  <xacro:property name="base_length" value="0.24" />
-  <xacro:property name="base_width" value="0.275" />
-  <xacro:property name="base_height" value="0.003" />
+  <xacro:property name="base_length" value="0.30" />
+  <xacro:property name="base_width" value="0.26" />
+  <xacro:property name="base_height" value="0.08" />
   <xacro:property name="base_mass" value="1" />
-  <xacro:property name="wheel_radius" value="0.045" />
+  <xacro:property name="wheel_radius" value="0.05" />
   <xacro:property name="wheel_width" value="0.01" />
-  <xacro:property name="wheel_pos_x" value="0.0" />
+  <xacro:property name="wheel_pos_x" value="0.10" />
   <xacro:property name="wheel_pos_y" value="0.13" />
   <xacro:property name="wheel_pos_z" value="-0.03" />
   <xacro:property name="wheel_mass" value=".1" />
   <xacro:property name="wheel_torque" value="20" />
-  <xacro:property name="front_caster_wheel" value="true" />
+  <xacro:property name="front_caster_wheel" value="false" />
   <xacro:property name="rear_caster_wheel" value="true" />
   <xacro:property name="laser_pose">
-    <origin xyz="0.12 0 0.13" rpy="0 0 0"/>
+    <origin xyz="0.10 0 0.10" rpy="0 0 0"/>
   </xacro:property>
   <xacro:property name="depth_sensor_pose">

Commit message: MARRtino ROS2

File: marrtinorobot2_description/urdf/2wd_properties.urdf.xacro (robot description, xacro)
@@ -5,6 +5,6 @@
   <xacro:property name="base_height" value="0.08" />
   <xacro:property name="base_mass" value="1" />
-  <xacro:property name="wheel_radius" value="0.05" />
-  <xacro:property name="wheel_width" value="0.01" />
+  <xacro:property name="wheel_radius" value="0.07" />
+  <xacro:property name="wheel_width" value="0.02" />
   <xacro:property name="wheel_pos_x" value="0.10" />
   <xacro:property name="wheel_pos_y" value="0.13" />
