Commit message: 4WD Urdf

File: marrtinorobot2_description/urdf/4wd_properties.urdf.xacro (robot description, xacro)
@@ -1,20 +1,20 @@
 <?xml version="1.0"?>
 <robot xmlns:xacro="http://ros.org/wiki/xacro">
-  <xacro:property name="base_length" value="0.445" />
-  <xacro:property name="base_width" value="0.200" />
-  <xacro:property name="base_height" value="0.129" />
+  <xacro:property name="base_length" value="0.275" />
+  <xacro:property name="base_width" value="0.160" />
+  <xacro:property name="base_height" value="0.08" />
   <xacro:property name="base_mass" value="10" />
-  <xacro:property name="wheel_radius" value="0.07162" />
+  <xacro:property name="wheel_radius" value="0.065" />
   <xacro:property name="wheel_width" value="0.05" />
-  <xacro:property name="wheel_pos_x" value="0.120" />
-  <xacro:property name="wheel_pos_y" value="0.1355" />
+  <xacro:property name="wheel_pos_x" value="0.085" />
+  <xacro:property name="wheel_pos_y" value="0.12" />
   <xacro:property name="wheel_pos_z" value="-0.04788" />
   <xacro:property name="wheel_mass" value=".6" />
   <xacro:property name="wheel_torque" value="20" />
   <xacro:property name="laser_pose">
-    <origin xyz="-0.0475 0 0.125" rpy="0 0 0"/>
+    <origin xyz="0 0 0.10" rpy="0 0 0"/>
   </xacro:property>
   <xacro:property name="depth_sensor_pose">
-    <origin xyz="-0.065 0 0.255" rpy="0 0 0"/>
+    <origin xyz="0.15 0 0.02" rpy="0 0 0"/>
   </xacro:property>
 </robot>
