Commit message: Update Gazebo

File: marrtinorobot2_description/urdf/marrtino_properties.urdf.xacro (robot description, xacro)
@@ -3,5 +3,5 @@
   <xacro:property name="base_length" value="0.49" />
   <xacro:property name="base_width" value="0.43" />
-  <xacro:property name="base_height" value="0.17" />
+  <xacro:property name="base_height" value="0.15" />
   <xacro:property name="base_mass" value="1" />
   <xacro:property name="wheel_radius" value="0.075" />
